File: thermometer.sch (KiCad schematic (older format))
At the start: 47 parts, among them J1 Display, J2 USB, J3 Battery, J4 Programming, J5 DS18B20, SW1 SW_Push, U1 STM32F072CBTx, U2 MCP73831-2-OT, U3 TPS2115, U4 LDS3985M33R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

Commit message: Changed button and dcdc placements
Changed lines of the file:
@@
 EESchema Schematic File Version 4
 LIBS:thermometer-cache
-EELAYER 29 0
+EELAYER 30 0
 EELAYER END
 $Descr A3 16535 11693
@@
 	2850 8300 2400 8300
 Connection ~ 2850 8300
-Text Label 8500 6200 0    50   ~ 0
+Text Label 8500 6100 0    50   ~ 0
 POW_STAT
 Wire Wire Line
@@
 	1    0    0    -1
 $EndComp
-Text Label 8500 6100 0    50   ~ 0
+Text Label 8500 6200 0    50   ~ 0
 CHG_STAT
 Wire Wire Line
